File: ROSBoardMini.sch (KiCad schematic (older format))
At the start: 61 parts, among them J1 Conn_02x20_Odd_Even, J2 Extension0, J3 Extension1, J4 Extension2, J5 PWR, J6 Extension2, U1 P2X8C4M64P, U10 LY68L6400SLIT, U2 W25Q128JVS, U3 PCA9544APW, U4 BME280, U5 ICM-20948, U6 24LC256, U7 AZ1117-1.8, U8 AZ1117-1.2, U9 AZ1117-2.85, Y1 Crystal_GND23

Commit message: Rooting done
Parts:
- removed C16, C21: 4.7uF, Capacitor_SMD:C_0402_1005Metric, symbol ROSBoardMini-rescue:C-Device
Other:
- moved on the sheet: C14, C23
Changed lines of the file:
@@
 L ROSBoardMini-rescue:C-Device C14
 U 1 1 5FB9C3CF
-P 3450 5650
-F 0 "C14" H 3565 5696 50  0000 L CNN
-F 1 "4.7uF" H 3565 5605 50  0000 L CNN
-F 2 "Capacitor_SMD:C_0402_1005Metric" H 3488 5500 50  0001 C CNN
-F 3 "~" H 3450 5650 50  0001 C CNN
-	1    3450 5650
+P 3900 5650
+F 0 "C14" H 4015 5696 50  0000 L CNN
+F 1 "4.7uF" H 4015 5605 50  0000 L CNN
+F 2 "Capacitor_SMD:C_0402_1005Metric" H 3938 5500 50  0001 C CNN
+F 3 "~" H 3900 5650 50  0001 C CNN
+	1    3900 5650
 	1    0    0    -1
 $EndComp
@@
 $EndComp
 $Comp
-L ROSBoardMini-rescue:C-Device C16
-U 1 1 5FBA5477
-P 3900 5650
-F 0 "C16" H 4015 5696 50  0000 L CNN
-F 1 "4.7uF" H 4015 5605 50  0000 L CNN
-F 2 "Capacitor_SMD:C_0402_1005Metric" H 3938 5500 50  0001 C CNN
-F 3 "~" H 3900 5650 50  0001 C CNN
-	1    3900 5650
-	1    0    0    -1
-$EndComp
-$Comp
 L ROSBoardMini-rescue:C-Device C19
 U 1 1 5FBA75EC
@@
 $EndComp
 $Comp
-L ROSBoardMini-rescue:C-Device C21
-U 1 1 5FBA75F2
+L ROSBoardMini-rescue:C-Device C23
+U 1 1 5FBAAD71
 P 4800 5650
-F 0 "C21" H 4915 5696 50  0000 L CNN
+F 0 "C23" H 4915 5696 50  0000 L CNN
 F 1 "4.7uF" H 4915 5605 50  0000 L CNN
 F 2 "Capacitor_SMD:C_0402_1005Metric" H 4838 5500 50  0001 C CNN
@@
 	1    0    0    -1
 $EndComp
-$Comp
-L ROSBoardMini-rescue:C-Device C23
-U 1 1 5FBAAD71
-P 5250 5650
-F 0 "C23" H 5365 5696 50  0000 L CNN
-F 1 "4.7uF" H 5365 5605 50  0000 L CNN
-F 2 "Capacitor_SMD:C_0402_1005Metric" H 5288 5500 50  0001 C CNN
-F 3 "~" H 5250 5650 50  0001 C CNN
-	1    5250 5650
-	1    0    0    -1
-$EndComp
-Wire Wire Line
-	5250 5500 4800 5500
-Connection ~ 3900 5500
-Wire Wire Line
-	3900 5500 3450 5500
 Connection ~ 4350 5500
-Wire Wire Line
-	4350 5500 3900 5500
-Connection ~ 4800 5500
-Wire Wire Line
-	4800 5500 4350 5500
-Wire Wire Line
-	3450 5800 3900 5800
-Connection ~ 3900 5800
-Wire Wire Line
-	3900 5800 4350 5800
 Connection ~ 4350 5800
-Wire Wire Line
-	4350 5800 4800 5800
-Connection ~ 4800 5800
-Wire Wire Line
-	4800 5800 5250 5800
 $Comp
 L ROSBoardMini-rescue:+1V8-power #PWR0191
@@
 NoConn ~ 13150 3800
 NoConn ~ 8250 3800
+Wire Wire Line
+	4350 5500 4800 5500
+Wire Wire Line
+	4350 5800 4800 5800
+Wire Wire Line
+	3900 5500 4350 5500
+Wire Wire Line
+	3900 5800 4350 5800
 $EndSCHEMATC

Commit message: Clean schematic and rename 4th connector
Parts:
- J6: value Extension2 -> Extension3
Other:
- note added: "Barometer"
- note added: "Extension port compatible with the OV2640\n with only Parallax Propeller 2 IO"
- note added: "Extension port with a mix of\nPi Zero IO and P2 IO"
- note added: "Flash memory"
- note added: "I2C Multiplexer"
- note added: "IMU"
- note added: "PSRAM"
- note added: "Parallax Propeller 2"
- note added: "Pi Zero"
- note added: "Power"
- note added: "Sensor"
- note removed: "TODO\nCheck vi/vo for 3.3v/2.8v"
- moved on the sheet: C10, C11, C12, C13, C14, C15, C17, C18, C19, C20, C22, C23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

Commit message: Various cleaning, doc in schematic and replaced problematic 2.8V ldo
Parts:
- removed U9: AZ1117-2.85, Package_TO_SOT_SMD:SOT-89-3, symbol ROSBoardMini-rescue:AZ1117-2.85-Regulator_Linear
- added C1: 0.1uF, Capacitor_SMD:C_0402_1005Metric, symbol Device:C
- added U9: MIC5353-2.8YMT, Package_DFN_QFN:MLF-6-1EP_1.6x1.6mm_P0.5mm_EP0.5x1.26mm, symbol Regulator_Linear:MIC5353-2.8YMT
- C13, C18, C31, C7, C8, C9: value 100nF -> 0.1uF
- C27: value 10uF -> 1uF
- C30: value 22uF -> 1uF
Connections:
- net +2V8: now also U9.4 (VOUT)
- net +3V3: now also U9.1 (EN), U9.3 (VIN)
- net GND: now also C1.2, U9.2 (GND), U9.7 (GND)
- new net: C1.1, U9.6 (BYP)
Other:
- moved on the sheet: C25, C26, C27, C28, C29, C30, C8, U7, U8

Commit message: Add crystal reference
Parts:
- Y1: value Crystal_GND23 -> ABM8-25.000MHZ-10-D1G-T
Changed lines of the file:
@@
 P 1000 3650
 F 0 "Y1" V 550 3650 50  0000 L CNN
-F 1 "Crystal_GND23" V 650 3400 50  0000 L CNN
+F 1 "ABM8-25.000MHZ-10-D1G-T" V 650 3400 50  0000 L CNN
 F 2 "Crystal:Crystal_SMD_Abracon_ABM8G-4Pin_3.2x2.5mm" H 1000 3650 50  0001 C CNN
 F 3 "~" H 1000 3650 50  0001 C CNN
